File: Commodore-Vic-20.sch (KiCad schematic (older format))
At the start: 144 parts, among them CN1 Conn_01x03_Female, CN2 Conn_01x03_Male, P1 User Port, P10 Keyboard, P2 CONN_Cassette, P3 Serial, P4 Audio / Video, P5 Controller Port, P6 Expansion Port, P7 Power, Q1 2SC1815, Q2 2SC1959, Q3 2SC1815, Q4 2SD880, SW1 SW_DPST, U13 74LS08, U14 M58725, U15 M58725, Y1 14.31818

Commit message: Use 6502 from Kicad library
Parts:
- removed UE10: 6502, Package_DIP:DIP-40_W15.24mm, symbol Commodore-Vic-20:6502
- added UE10: 6502, Package_DIP:DIP-40_W15.24mm, symbol CPU_Obsolete:6502
Connections:
- wire segments 1129 -> 1130
Other:
- moved on the sheet: C1
